File: Modules/Module 1/555Board/555Board.kicad_pcb (KiCad board)
At the start: 2 copper layers, 44.5 x 16.2 mm, 10 parts, among them J1 Barrel Jack, J2 2.54mm 1x2 Header, U1 LM555xM

Commit message: Module 2 Done
Parts:
- removed J1: Barrel Jack, Connector_BarrelJack:BarrelJack_GCT_DCJ200-10-A_Horizontal
- J2: footprint Connector_PinHeader_2.54mm:PinHeader_1x02_P2.54mm_Vertical -> Connector_PinHeader_2.54mm:PinHeader_1x02_P2.54mm_Vertical_SMD_Pin1Left
- moved J2 6.58 mm to (163.5, 69.0)
- moved R3 1.72 mm to (192.8, 64.2), turned to 90 degrees
Connections:
- R3 pad 2: 9V0 -> GND
Routing:
- net 9V0: track 44.4 -> 27.0 mm
- net GND: track 28.9 -> 33.5 mm
- net Net-(U1-THRES): track 52.9 -> 48.8 mm
- net Net-(D2-A): track 30.1 -> 27.8 mm
- net Net-(D2-K): track 3.62 -> 2.82 mm
Other:
- board size 44.5 x 16.2 mm -> 35.8 x 15.2 mm

Commit message: Plenty of updates
Parts:
- added G***: LOGO, LOGO, F.Cu at (177.5, 61.6)
- added G***: LOGO, LOGO, F.Cu at (167.3, 61.5)
Other:
- board size 35.8 x 15.2 mm -> 35.8 x 17.7 mm
- board text added: "555 Timer Board"
- board text added: "9V"
- board text added: "GND"
