File: Modules/Module 2/FTDIBoard/FTDIBoard.kicad_sch (KiCad schematic)
At the start: 13 parts, among them J1 USB_C_Receptacle_USB2.0_16P, J3 Conn_01x03, U1 FT232RL

Commit message: edits
Other:
- note added: "**Make sure MCU is running at 5V"
Changed lines of the file:
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@@
 	(generator_version "10.0")
 	(paper "A4")
+	(text "**Make sure MCU is running at 5V"
+		(exclude_from_sim no)
+		(at 185.42 65.024 0)
+		(effects
+			(font
+				(size 1.27 1.27)
+			)
+			(justify left)
+		)
+	)
 	(text "5V\nUPDI\nGND"
 		(exclude_from_sim no)
