File: Modules/Module 2/FTDIBoard/FTDIBoard.kicad_pcb (KiCad board)
At the start: 2 copper layers, 38.8 x 17.2 mm, 13 parts, among them J1 USB_C_Receptacle_USB2.0_16P, J3 Conn_01x03, U1 FT232RL

Commit message: Plenty of updates
Parts:
- added G***: LOGO, LOGO, F.Cu at (153.1, 89.0)
- added G***: LOGO, LOGO, F.Cu at (174.2, 89.2)
Other:
- board size 38.8 x 17.2 mm -> 38.8 x 21.8 mm
- board text added: "5V"
- board text added: "FTDI Programmer Board"
- board text added: "GND"
- board text added: "UPDI"
