File: Modules/Module 2/ATtinyBoard/ATtinyBoard.kicad_pcb (KiCad board)
At the start: 2 copper layers, 26.2 x 14.8 mm, 6 parts, among them J1 Conn_01x03, SW1 SW_Push, U1 ATtiny412-SS

Commit message: Plenty of updates
Parts:
- added G***: LOGO, LOGO, F.Cu at (162.2, 109.8)
- added G***: LOGO, LOGO, F.Cu at (143.4, 109.8)
Other:
- board size 26.2 x 14.8 mm -> 29.8 x 18.8 mm
- board text added: "5V0"
- board text added: "ATtiny412 Board"
- board text added: "GND"
- board text added: "UPDI"
