File: Modules/Module 3/SEEEDXIAOESP32C6_Basic/SEEEDXIAOESP32C6_Basic.kicad_pcb (KiCad board)
At the start: 2 copper layers, 29.2 x 21.5 mm, 5 parts, among them J1 Conn_01x07_Socket, J2 Conn_01x07_Socket, SW1 SW_Push

Commit message: Plenty of updates
Parts:
- added G***: LOGO, LOGO, F.Cu at (132.1, 102.6)
- added G***: LOGO, LOGO, F.Cu at (128.4, 93.5)
Other:
- board size 29.2 x 21.5 mm -> 34.8 x 25.5 mm
- board text added: "Basic Board"
- board text added: "ESP32 C6"
- board text added: "SEEED XIAO"
