File: Modules/Module 4/SEEEDXIAOESP32C6_Accelerometer/SEEEDXIAOESP32C6_Accelerometer.kicad_pcb (KiCad board)
At the start: 2 copper layers, 38.2 x 27.2 mm, 9 parts, among them J1 Conn_01x07_Socket, J2 Conn_01x07_Socket, U1 BMI270

Commit message: Plenty of updates
Parts:
- added G***: LOGO, LOGO, F.Cu at (138.7, 105.7)
- added G***: LOGO, LOGO, F.Cu at (128.4, 103.7)
Other:
- board size 38.2 x 27.2 mm -> 38.2 x 28.1 mm
- board text added: "Accelerometer"
- board text added: "BMI270"
- board text added: "Board"
- board text added: "ESP32 C6"
- board text added: "SEEED XIAO"
