File: Modules/Module 5/SEEEDXIAOESP32C6_DCDriver/SEEEDXIAOESP32C6_DCDriver.kicad_pcb (KiCad board)
At the start: 2 copper layers, 47 x 22.8 mm, 8 parts, among them J1 Conn_01x07_Socket, J2 Conn_01x07_Socket, J3 Conn_01x02_Pin, J5 Conn_01x04_Pin, U1 TB6612FNG

Commit message: Plenty of updates
Parts:
- added G***: LOGO, LOGO, F.Cu at (136.1, 102.1)
- added G***: LOGO, LOGO, F.Cu at (126.3, 102.1)
Routing:
- net /BDIR1: track 40.7 -> 33.6 mm
Other:
- board size 47 x 22.8 mm -> 47 x 25.3 mm
- board text added: "DC & Stepper Motor Driver Board"
- board text added: "ESP32 C6"
- board text added: "SEEED XIAO"
