File: Modules/Module 7/SEEEDXIAOESP32C6_Neopixel/SEEEDXIAOESP32C6_Neopixel.kicad_pcb (KiCad board)
At the start: 2 copper layers, 34.8 x 23.2 mm, 5 parts, among them J1 Conn_01x07_Socket, J2 Conn_01x07_Socket

Commit message: Plenty of updates
Parts:
- added C2: 0.1uF, Capacitor_SMD:C_1206_3216Metric_Pad1.33x1.80mm_HandSolder, F.Cu at (129.9, 98.9)
- added D3: WS2812B, LED_SMD:LED_WS2812B_PLCC4_5.0x5.0mm_P3.2mm, F.Cu at (130.0, 103.0)
- added G***: LOGO, LOGO, F.Cu at (132.2, 84.9)
- added G***: LOGO, LOGO, F.Cu at (136.2, 99.0)
Connections:
- D2 pad 2: unconnected-(D2-DOUT-Pad2) -> Net-(D2-DOUT)
Routing:
- net 3V3: track 37.0 -> 48.3 mm
- net Net-(D2-DOUT): track 0.00 -> 9.16 mm
- net GND: vias 2 -> 4
Other:
- board size 34.8 x 23.2 mm -> 34.8 x 26.4 mm
- board text added: "ESP32 C6"
- board text added: "Neopixel Board"
- board text added: "SEEED XIAO"
