File: Modules/Module 7/SEEEDXIAOESP32C6_Neopixel/SEEEDXIAOESP32C6_Neopixel.kicad_sch (KiCad schematic)
At the start: 5 parts, among them J1 Conn_01x07_Socket, J2 Conn_01x07_Socket

Commit message: Plenty of updates
Parts:
- added C2: 0.1uF, Capacitor_SMD:C_1206_3216Metric_Pad1.33x1.80mm_HandSolder, symbol Device:C
- added D3: WS2812B, LED_SMD:LED_WS2812B_PLCC4_5.0x5.0mm_P3.2mm, symbol LED:WS2812B
Connections:
- net 3V3: now also C2.1, D3.1 (VDD)
- net GND: now also C2.2, D3.3 (VSS)
- net at D2.2 (DOUT): now also D3.4 (DIN)
Other:
- moved on the sheet: C1
