File: Modules/Analog & Digital Servo Tester/ServoTesterBoard/ServoTesterBoard.kicad_pcb (KiCad board)
At the start: 2 copper layers, 70.5 x 41.1 mm, 24 parts, among them J1 Barrel Jack, J2 2.54mm 1x2 Header, J3 2.54mm 1x3 Header, Q1 BC547, SW1 Slide Switch, SW2 Push Button, SW3 Push Button, U1 LM555xM, U2 L7805

Commit message: Analog & Digital Servo Tester Added
Parts:
- added G***: LOGO, LOGO, F.Cu at (185.5, 65.0)
- added G***: LOGO, LOGO, F.Cu at (167.5, 64.8)
Other:
- board text removed: "Designed by:"
- board text removed: "Nicholas Niles"
- board text removed: "https://nicholasniles.com/"
