File: Modules/LiPoBMS/LiPoBMS.kicad_sch (KiCad schematic)
At the start: 8 parts, among them J1 Conn_01x02_Pin, J2 Conn_01x02_Pin, U1 MCP73831T-2ACI/OT

Commit message: Firmware Work
Other:
- note added: "(https://cdn.sparkfun.com/datasheets/Components/General%20IC/33244_SPCN.pdf)"
- note added: "33k used in Demo for 40mAh cell"
- note added: "See page 7 of datasheet:"
Changed lines of the file:
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@@
+		)
+	)
+	(text "(https://cdn.sparkfun.com/datasheets/Components/General%20IC/33244_SPCN.pdf)"
+		(exclude_from_sim no)
+		(at 247.142 109.728 0)
+		(effects
+			(font
+				(size 1.016 1.016)
+			)
+		)
+	)
+	(text "See page 7 of datasheet: "
+		(exclude_from_sim no)
+		(at 227.076 107.696 0)
+		(effects
+			(font
+				(size 1.27 1.27)
+			)
+		)
+	)
+	(text "33k used in Demo for 40mAh cell"
+		(exclude_from_sim no)
+		(at 230.886 99.314 0)
+		(effects
+			(font
+				(size 1.27 1.27)
+			)
 		)
 	)
